File: PCB/HexadecipadV2/HexadecipadV2.kicad_sch (KiCad schematic)
At the start: 88 parts, among them SW1 Encoder, SW10 SW_Push_45deg, SW11 SW_Push_45deg, SW12 SW_Push_45deg, SW13 SW_Push_45deg, SW14 SW_Push_45deg, SW15 SW_Push_45deg, SW16 SW_Push_45deg, SW17 SW_Push_45deg, SW18 SW_Push_45deg, SW19 SW_Push_45deg, SW2 Encoder, SW20 SW_Push_45deg, SW21 SW_Push_45deg, SW22 SW_Push_45deg, SW23 SW_Push_45deg, SW24 SW_Push_45deg, SW25 SW_Push_45deg, SW26 SW_Push_45deg, SW27 SW_Push_45deg, SW28 SW_Push_45deg, SW3 Encoder, SW4 Encoder, SW5 SW_Push_45deg, SW6 SW_Push_45deg, SW7 SW_Push_45deg, SW8 SW_Push_45deg, SW9 SW_Push_45deg, U1 XIAO-RP2040-DIP, U2 MCP23017_SP, U3 MCP23017_SP

Commit message: Fix all traces
I stopped using freerouting because i realised it was not allowed and it was a huge pain. redid all the traces by hand and made some power planes. removed all of my LEDs because 1.21 GIGAWATTS
Parts:
- removed D29, D30, D31, D32, D33, D34, D35, D36, D37, D38, D39, D40, D41, D42, D43, D44, D45, D46, D47, D48, D49, D50, D51, D52: SK6812MINI, kicad-keyboard-parts.pretty-master:MX_SK6812MINI-E_REV, symbol LED:SK6812MINI
- removed R3, R4, R5: R, Resistor_THT:R_Axial_DIN0207_L6.3mm_D2.5mm_P7.62mm_Horizontal, symbol Device:R
- removed U3: MCP23017_SP, Package_DIP:DIP-28_W7.62mm, symbol Interface_Expansion:MCP23017_SP
Connections:
- net LEDs is gone; now on net ENC3-A: U1.11 (GPIO3/MOSI)
- net Column 0: now also U2.7 (GPB6); no longer SW25.1, U2.21 (GPA0)
- net Column 1: now also U2.8 (GPB7); no longer SW26.1, U2.22 (GPA1)
- net Column 2: no longer SW27.1
- net Column 3: now also U2.22 (GPA1); no longer SW28.1, U2.24 (GPA3)
- net ENC1-A: now also U1.4 (GPIO29/ADC3/A3); no longer U2.25 (GPA4)
- net ENC1-B: now also U1.3 (GPIO28/ADC2/A2); no longer U2.26 (GPA5)
- net ENC2-A: now also U1.2 (GPIO27/ADC1/A1); no longer U2.27 (GPA6)
- net ENC2-B: now also U1.1 (GPIO26/ADC0/A0); no longer U2.28 (GPA7)
- net ENC3-B: now also U1.10 (GPIO4/MISO)
- net ENC4-A: now also U1.9 (GPIO2/SCK)
- net ENC4-B: now also U1.8 (GPIO1/RX)
- net Row 1: now also D24.1 (K)
- net Row 2: now also D23.1 (K)
- net Row 3: now also D22.1 (K)
- net Row 4: now also D21.1 (K)
- net SCK MCP: now also U1.6 (GPIO7/SCL); no longer U1.9 (GPIO2/SCK)
- net SDA MCP: now also U1.5 (GPIO6/SDA); no longer U1.8 (GPIO1/RX)
- net 5V: no longer names the net of U1.14 (VBUS)
- removed net Row 6: D21.1 (K), D22.1 (K), D23.1 (K), D24.1 (K), U2.7 (GPB6)
- new net Column 4: SW25.1, SW26.1, SW27.1, SW28.1, U2.21 (GPA0)
- no-connect marks 5 -> 9
Other:
- moved on the sheet: D21, D22, D23, D24, SW25, SW26, SW27, SW28
